File: Examples/Half_Adder/half_adder.sch (KiCad schematic (older format))
At the start: 3 parts, among them U1 PORT, U2 d_xor, U3 d_and

Commit message: ngspice issue resolved
Connections:
- wire segments 12 -> 14
Changed lines of the file:
@@
-EESchema Schematic File Version 2
+EESchema Schematic File Version 4
 LIBS:power
 LIBS:device
-LIBS:transistors
-LIBS:conn
-LIBS:linear
-LIBS:regul
 LIBS:74xx
-LIBS:cmos4000
-LIBS:adc-dac
-LIBS:memory
-LIBS:xilinx
-LIBS:special
-LIBS:microcontrollers
-LIBS:dsp
-LIBS:microchip
-LIBS:analog_switches
-LIBS:motorola
-LIBS:texas
-LIBS:intel
 LIBS:audio
 LIBS:interface
-LIBS:digital-audio
-LIBS:philips
-LIBS:display
-LIBS:cypress
-LIBS:siliconi
-LIBS:opto
-LIBS:atmel
-LIBS:contrib
-LIBS:valves
-LIBS:eSim_Analog
-LIBS:eSim_Devices
-LIBS:eSim_Digital
-LIBS:eSim_Hybrid
-LIBS:eSim_Sources
-LIBS:eSim_Subckt
-EELAYER 25 0
+LIBS:Half_Adder-cache
+EELAYER 29 0
 EELAYER END
 $Descr A4 11693 8268
@@
 $EndComp
 Wire Wire Line
-	5200 2950 4450 2950
+	5200 2950 5000 2950
 Wire Wire Line
 	4450 2950 4450 3000
@@
 	4550 3450 4550 3050
 Wire Wire Line
-	4550 3050 5200 3050
+	4550 3050 4850 3050
 Wire Wire Line
 	5250 3700 5000 3700
@@
 Text Notes 6200 3650 0    60   ~ 0
 COUT\n
+Wire Wire Line
+	5000 2950 4450 2950
+Wire Wire Line
+	4850 3050 5200 3050
 $EndSCHEMATC
