File: Examples/HalfAdder/half_adder.sch (KiCad schematic (older format))
At the start: 3 parts, among them U1 PORT, U2 d_xor, U3 d_and

Commit message: examples
Parts:
- removed U1: PORT, symbol PORT
- removed U2: d_xor, symbol d_xor
- removed U3: d_and, symbol d_and
- added R1, R2: 1k, symbol R
- added U1: adc_bridge_2, symbol adc_bridge_2
- added U2: dac_bridge_2, symbol dac_bridge_2
- added U3, U4, U5, U6: plot_v1, symbol plot_v1
- added X1: half_adder, symbol half_adder
- added v1, v2: DC, R1, symbol DC
Connections:
- net labels added: GND, IN1, IN2, cout, sum
- wire segments 12 -> 37
Other:
- note removed: "COUT\n"
- note removed: "IN1\n\n"
- note removed: "IN2"
- note removed: "SUM\n"
